File: KiCad_Project/Audio_Amp_v1/.history/Audio_Amp_v1.kicad_pcb (KiCad board)
At the start: 2 copper layers, 93.5 x 52.8 mm, 73 parts, among them IC2 TPA3116D2DAD, IC3 BM64SPKS1MC2-0002AA, IC4 LMR33630ADDA, J1 TS-103-T-A, J2 1729128, J3 1729128, J4 PJ-102AH

Commit message: added logo
Other:
- board text removed: "Loredati_svg"
