File: KiCad_Project/Audio_Amp_v1/05_Power_Amplifier.kicad_sch (KiCad schematic)
At the start: 43 parts, among them IC2 TPA3116D2DAD

Commit message: added gerber files, csv and BOM_pos
Parts:
- C1, C2, C3, C4, C5: LCSC (none) -> C5199872
- C10, C17: LCSC (none) -> C116211
- C11, C12, C13, C14: LCSC (none) -> C5378
- C15, C8: LCSC (none) -> C46653
- C16, C9: LCSC (none) -> C49678
- C18, C19, C24, C25: LCSC (none) -> C1881
- C20, C21, C26, C27: LCSC (none) -> C100040
- C22, C23, C28, C29, C6: LCSC (none) -> C100042
- C7: LCSC (none) -> C1591
- IC2: LCSC (none) -> C50144
- R1, R3, R4: LCSC (none) -> C2907088
- R2: LCSC (none) -> C25586
- R5, R6, R7, R8, R9: LCSC (none) -> C2907471
