File: KiCad_Project/Audio_Amp_v1/Audio_Amp_v1.kicad_pcb (KiCad board)
At the start: 2 copper layers, 93.5 x 52.8 mm, 73 parts, among them IC2 TPA3116D2DAD, IC3 BM64SPKS1MC2-0002AA, IC4 LMR33630ADDA, J1 TS-103-T-A, J2 1729128, J3 1729128, J4 PJ-102AH

Commit message: DRC clean and layout fix
Routing:
- net GNDA: track 63.1 -> 61.2 mm, vias 73 -> 81
- net +3.3V: vias 15 -> 18
