File: KiCad_Project/Audio_Amp_v1/Audio_Amp_v1.kicad_pcb (KiCad board)
At the start: 4 copper layers, 102 x 64 mm, 124 parts, among them IC2 TPA3116D2DAD, J1 Screw_Terminal_01x02, J2 Screw_Terminal_01x02, J3 Barrel_Jack_Switch, J6 USB_C_Receptacle_USB2.0_16P, Q1 Q_PMOS_GDS, Q2 BSS138, U1 PCM2704CDB, U2 USBLC6-2SC6, U3 OPA1678IDR, U4 L78L12_SOT89

Commit message: layout corrections
Parts:
- renumbered TP3 to 12V, TP4 to 24V, 12V to D2, VBUS to D3, PLAY to D4
Changed lines of the file:
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@@
 		(descr "SMD pad as test Point, diameter 2.0mm")
 		(tags "test point SMD pad")
-		(property "Reference" "TP4"
+		(property "Reference" "24V"
 			(at 0 -1.998 0)
 			(layer "F.SilkS")
@@
 		(descr "SMD pad as test Point, diameter 2.0mm")
 		(tags "test point SMD pad")
-		(property "Reference" "TP3"
+		(property "Reference" "12V"
 			(at 0 -1.998 0)
 			(layer "F.SilkS")
@@
 		(descr "LED SMD 0805 (2012 Metric), square (rectangular) end terminal, IPC-7351 nominal, (Body size source: https://docs.google.com/spreadsheets/d/1BsfQQcO9C6DZCsRaXUlFlo91Tg2WpOkGARC1WS5S8t0/edit?usp=sharing)")
 		(tags "LED")
-		(property "Reference" "VBUS"
+		(property "Reference" "D3"
 			(at -0.2 -1.65 90)
 			(layer "F.SilkS")
@@
 		(descr "LED SMD 0805 (2012 Metric), square (rectangular) end terminal, IPC-7351 nominal, (Body size source: https://docs.google.com/spreadsheets/d/1BsfQQcO9C6DZCsRaXUlFlo91Tg2WpOkGARC1WS5S8t0/edit?usp=sharing)")
 		(tags "LED")
-		(property "Reference" "12V"
+		(property "Reference" "D2"
 			(at -3 0 0)
 			(layer "F.SilkS")
@@
 			(pinfunction "SHIELD_SH")
 			(pintype "passive")
+			(zone_connect 1)
 			(teardrops
 				(best_length_ratio 0.5)
@@
 			(pinfunction "SHIELD_SH")
 			(pintype "passive")
+			(zone_connect 1)
 			(teardrops
 				(best_length_ratio 0.5)
@@
 			(pinfunction "SHIELD_SH")
 			(pintype "passive")
+			(zone_connect 1)
 			(teardrops
 				(best_length_ratio 0.5)
@@
 			(pinfunction "SHIELD_SH")
 			(pintype "passive")
+			(zone_connect 1)
 			(teardrops
 				(best_length_ratio 0.5)
@@
 		(descr "LED SMD 0805 (2012 Metric), square (rectangular) end terminal, IPC-7351 nominal, (Body size source: https://docs.google.com/spreadsheets/d/1BsfQQcO9C6DZCsRaXUlFlo91Tg2WpOkGARC1WS5S8t0/edit?usp=sharing)")
 		(tags "LED")
-		(property "Reference" "PLAY"
+		(property "Reference" "D4"
 			(at 2.2 0 180)
 			(layer "F.SilkS")
@@
 		(start 119.8 84.8)
 		(end 119.8 91.35)
-		(width 0.6)
+		(width 0.8)
 		(layer "F.Cu")
 		(net "+24V")
@@
 		(start 105.4625 84.4)
 		(end 105.4625 86.7625)
-		(width 0.2)
+		(width 0.3)
 		(layer "F.Cu")
 		(net "+12V")
@@
 	)
 	(segment
-		(start 103.375 88.875)
+		(start 103.5 89.8)
 		(end 103.375 89.925)
 		(width 0.2)
@@
 	)
 	(segment
-		(start 103.5 89.8)
-		(end 103.375 89.925)
+		(start 102.905 88.605)
+		(end 103.375 89.075)
 		(width 0.2)
 		(layer "F.Cu")
@@
 	)
 	(segment
-		(start 98.04241 88.605)
-		(end 103.105 88.605)
+		(start 103.375 89.075)
+		(end 103.375 89.925)
 		(width 0.2)
 		(layer "F.Cu")
@@
 	)
 	(segment
-		(start 103.105 88.605)
-		(end 103.375 88.875)
+		(start 98.04241 88.605)
+		(end 102.905 88.605)
 		(width 0.2)
 		(layer "F.Cu")
@@
 		(layer "F.Cu")
 		(hatch none 0.1)
-		(priority 30013)
+		(priority 30000)
 		(attr
 			(teardrop
@@
 		(layer "F.Cu")
 		(hatch none 0.1)
-		(priority 30083)
+		(priority 30002)
 		(attr
 			(teardrop
@@
 		(polygon
 			(pts
-				(xy 105.5625 86.202567) (xy 105.3625 86.202567) (xy 105.2 86.601569) (xy 105.4625 86.803567) (xy 105.725 86.8)
+				(xy 105.6125 86.202567) (xy 105.3125 86.202567) (xy 105.2 86.601569) (xy 105.4625 86.803567) (xy 105.725 86.8)
 			)
 		)
@@
 		(layer "F.Cu")
 		(hatch none 0.1)
-		(priority 30021)
+		(priority 30001)
 		(attr
 			(teardrop
@@
 		(layer "B.Cu")
 		(hatch none 0.1)
-		(priority 30013)
+		(priority 30000)
 		(attr
 			(teardrop
@@
 		(layer "B.Cu")
 		(hatch none 0.1)
-		(priority 30017)
+		(priority 30001)
 		(attr
 			(teardrop
@@
 		(layer "B.Cu")
 		(hatch none 0.1)
-		(priority 30019)
+		(priority 30002)
 		(attr
 			(teardrop
@@
 		(layer "B.Cu")
 		(hatch none 0.1)
-		(priority 30020)
+		(priority 30003)
 		(attr
 			(teardrop

Commit message: added Images folder and changed some relative paths in the Kicad preferences
Parts:
- moved C28 4.37 mm to (151.0, 110.2), turned to 90 degrees
- moved C23 4.27 mm to (151.0, 92.2), turned to 90 degrees
- moved C29 4.27 mm to (151.0, 125.8), turned to 90 degrees
- moved C22 3.26 mm to (153.2, 109.2), turned to 0 degrees
- moved J1 1.50 mm to (160.4, 102.0)
- moved J2 1.50 mm to (160.4, 120.5)
- moved H1 1.41 mm to (158.0, 83.8)
- moved H2 1.41 mm to (158.0, 134.8)
- moved H3 1.41 mm to (69.0, 134.8)
- moved H4 1.41 mm to (69.0, 83.8), turned to 90 degrees
- moved J6 0.75 mm to (67.1, 93.2)
- moved R31 0.75 mm to (73.5, 95.2)
- moved R32 0.75 mm to (73.5, 91.2)
- moved C26 0.10 mm to (151.0, 113.2)
- moved R8 0.10 mm to (153.0, 112.5)
- renumbered 12V to TP3, 24V to TP4
Routing:
- net GNDA: track 126.4 -> 123.6 mm, vias 65 -> 67
- net /USB_DAC/USB_D+: track 10.8 -> 10.3 mm
- net Net-(C22-Pad2): track 2.03 -> 2.59 mm
Other:
- board size 102 x 64 mm -> 99.8 x 64 mm

Commit message: Use shared Kicad_Libs instead of project-specific libraries
- Project parts moved to Kicad_Libs (symbol, footprint, 3D, datasheet)
- Lib tables point to ${KIPRJMOD}/../KiCad_Libs (link via bring_libs.bat)
- Schematic/PCB references (lib ids, footprints, 3D paths, datasheets)
  updated to the Kicad_Libs libraries; no design changes
- Removed the old project-specific library folder
Parts:
- C10, C17: footprint EEE-FK1H221GV:EEHZT1E561UV -> eCapacitor:EEHZT1E561UV
- IC2: footprint TPA3116D2DAD:SOP65P810X120-32N -> eAmplifier:SOP65P810X120-32N
- L1, L2, L3, L4: footprint 7443341000:INDPM8479X720N -> eCoil:INDPM8479X720N
- U1: footprint PCM2704CDB:SOP65P780X200-28N -> eConverterADDA:SOP65P780X200-28N
Changed lines of the file:
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@@
 		)
 		(embedded_fonts no)
-		(model "C:/Users/lollo/Desktop/Hardware_Projects/Class-D-Bluetooth-5.0-Stereo-Audio-Amplifier/libs/Kicad_Library/Potentiometers/RK09712200HA.stp"
+		(model "${KIPRJMOD}/../KiCad_Libs/eResistor/eResistor.3dshapes/RK09712200HA.stp"
 			(offset
 				(xyz -4.5 -2.5 0.5)
@@
 		)
 	)
-	(footprint "TPA3116D2DAD:SOP65P810X120-32N"
+	(footprint "eAmplifier:SOP65P810X120-32N"
 		(layer "F.Cu")
 		(at 123 108.25)
@@
 			)
 		)
-		(property "Datasheet" "kicad-embed://tpa3116d2.pdf"
+		(property "Datasheet" "${KIPRJMOD}/../KiCad_Libs/eAmplifier/datasheet/tpa3116d2.pdf"
 			(at 0 0 0)
 			(layer "F.Fab")
@@
 		)
 		(embedded_fonts no)
-		(model "TPA3116D2DAD.stp"
+		(model "${KIPRJMOD}/../KiCad_Libs/eAmplifier/eAmplifier.3dshapes/TPA3116D2DAD.stp"
 			(offset
 				(xyz 0 0 0)
@@
 		)
 	)
-	(footprint "7443341000:INDPM8479X720N"
+	(footprint "eCoil:INDPM8479X720N"
 		(layer "F.Cu")
 		(at 142.5 113.5)
@@
 			)
 		)
-		(property "Datasheet" "kicad-embed://7443341000.pdf"
+		(property "Datasheet" "${KIPRJMOD}/../KiCad_Libs/eCoil/datasheet/7443341000.pdf"
 			(at 0 0 0)
 			(layer "F.Fab")
@@
 		)
 		(embedded_fonts no)
-		(model "7443341000.stp"
+		(model "${KIPRJMOD}/../KiCad_Libs/eCoil/eCoil.3dshapes/7443341000.stp"
 			(offset
 				(xyz 0 0 0.04999999999)
@@
 		)
 		(embedded_fonts no)
-		(model "C:/Users/lollo/Desktop/Hardware_Projects/Class-D-Bluetooth-5.0-Stereo-Audio-Amplifier/libs/Kicad_Library/Fuse/Littelfuse_2920L260_33DR.step"
+		(model "${KIPRJMOD}/../KiCad_Libs/eFuse/eFuse.3dshapes/Littelfuse_2920L260_33DR.step"
 			(offset
 				(xyz 0 0 0)
@@
 		)
 		(embedded_fonts no)
-		(model "C:/Users/lollo/Desktop/Hardware_Projects/Class-D-Bluetooth-5.0-Stereo-Audio-Amplifier/libs/Kicad_Library/Potentiometers/RK09L1220A1B.stp"
+		(model "${KIPRJMOD}/../KiCad_Libs/eResistor/eResistor.3dshapes/RK09L1220A1B.stp"
 			(offset
 				(xyz -2.5 -2.5 7)
@@
 		)
 	)
-	(footprint "7443341000:INDPM8479X720N"
+	(footprint "eCoil:INDPM8479X720N"
 		(layer "F.Cu")
 		(at 142.5 95.5)
@@
 			)
 		)
-		(property "Datasheet" "kicad-embed://7443341000.pdf"
+		(property "Datasheet" "${KIPRJMOD}/../KiCad_Libs/eCoil/datasheet/7443341000.pdf"
 			(at 0 0 0)
 			(layer "F.Fab")
@@
 		)
 		(embedded_fonts no)
-		(model "7443341000.stp"
+		(model "${KIPRJMOD}/../KiCad_Libs/eCoil/eCoil.3dshapes/7443341000.stp"
 			(offset
 				(xyz 0 0 0.04999999999)
@@
 		(embedded_fonts no)
 	)
-	(footprint "PCM2704CDB:SOP65P780X200-28N"
+	(footprint "eConverterADDA:SOP65P780X200-28N"
 		(layer "F.Cu")
 		(at 94.53741 92.18)
@@
 		)
 		(embedded_fonts no)
-		(model "C:/Users/lollo/Desktop/Hardware_Projects/Class-D-Bluetooth-5.0-Stereo-Audio-Amplifier/libs/Kicad_Library/DAC/PCM2704CDB/PCM2704CDB.STEP"
+		(model "${KIPRJMOD}/../KiCad_Libs/eConverterADDA/eConverterADDA.3dshapes/PCM2704CDB.STEP"
 			(offset
 				(xyz 0 0 0)
@@
 		)
 	)
-	(footprint "EEE-FK1H221GV:EEHZT1E561UV"
+	(footprint "eCapacitor:EEHZT1E561UV"
 		(layer "F.Cu")
 		(at 130.5 91)
@@
 			)
 		)
-		(property "Datasheet" "kicad-embed://ABA0000C1181.pdf"
+		(property "Datasheet" "${KIPRJMOD}/../KiCad_Libs/eCapacitor/datasheet/ABA0000C1181.pdf"
 			(at 0 0 0)
 			(layer "F.Fab")
@@
 		)
 		(embedded_fonts no)
-		(model "EEE-FK1H221GV.stp"
+		(model "${KIPRJMOD}/../KiCad_Libs/eCapacitor/eCapacitor.3dshapes/EEE-FK1H221GV.stp"
 			(offset
 				(xyz 0 0 0.999999985)
@@
 		)
 		(embedded_fonts no)
-		(model "C:/Users/lollo/Desktop/Hardware_Projects/Class-D-Bluetooth-5.0-Stereo-Audio-Amplifier/libs/Kicad_Library/Connectors/24V-JACK/PJ-102AH.stp"
+		(model "${KIPRJMOD}/../KiCad_Libs/eConnector/eConnector.3dshapes/PJ-102AH.stp"
 			(offset
 				(xyz 0 -13.5 7)
@@
 		)
 	)
-	(footprint "7443341000:INDPM8479X720N"
+	(footprint "eCoil:INDPM8479X720N"
 		(layer "F.Cu")
 		(at 142.5 122.5)
@@
 			)
 		)
-		(property "Datasheet" "kicad-embed://7443341000.pdf"
+		(property "Datasheet" "${KIPRJMOD}/../KiCad_Libs/eCoil/datasheet/7443341000.pdf"
 			(at 0 0 0)
 			(layer "F.Fab")
@@
 		)
 		(embedded_fonts no)
-		(model "7443341000.stp"
+		(model "${KIPRJMOD}/../KiCad_Libs/eCoil/eCoil.3dshapes/7443341000.stp"
 			(offset
 				(xyz 0 0 0.04999999999)
@@
 		)
 	)
-	(footprint "7443341000:INDPM8479X720N"
+	(footprint "eCoil:INDPM8479X720N"
 		(layer "F.Cu")
 		(at 142.5 104.5 180)
@@
 			)
 		)
-		(property "Datasheet" "kicad-embed://7443341000.pdf"
+		(property "Datasheet" "${KIPRJMOD}/../KiCad_Libs/eCoil/datasheet/7443341000.pdf"
 			(at 0 0 0)
 			(layer "F.Fab")
@@
 		)
 		(embedded_fonts no)
-		(model "7443341000.stp"
+		(model "${KIPRJMOD}/../KiCad_Libs/eCoil/eCoil.3dshapes/7443341000.stp"
 			(offset
 				(xyz 0 0 0.04999999999)
@@
 		)
 		(embedded_fonts no)
-		(model "C:/Users/lollo/Desktop/Hardware_Projects/Class-D-Bluetooth-5.0-Stereo-Audio-Amplifier/libs/Kicad_Library/Potentiometers/RK09L1220A1B.stp"
+		(model "${KIPRJMOD}/../KiCad_Libs/eResistor/eResistor.3dshapes/RK09L1220A1B.stp"
 			(offset
 				(xyz -2.5 -2.5 6.5)
@@
 		)
 	)
-	(footprint "EEE-FK1H221GV:EEHZT1E561UV"
+	(footprint "eCapacitor:EEHZT1E561UV"
 		(layer "F.Cu")
 		(at 130.5 124.25 180)
@@
 			)
 		)
-		(property "Datasheet" "kicad-embed://ABA0000C1181.pdf"
+		(property "Datasheet" "${KIPRJMOD}/../KiCad_Libs/eCapacitor/datasheet/ABA0000C1181.pdf"
 			(at 0 0 0)
 			(layer "F.Fab")
@@
 		)
 		(embedded_fonts no)
-		(model "EEE-FK1H221GV.stp"
+		(model "${KIPRJMOD}/../KiCad_Libs/eCapacitor/eCapacitor.3dshapes/EEE-FK1H221GV.stp"
 			(offset
 				(xyz 0 0 0.999999985)
