File: KiCad_Project/Audio_Amp_BT/01_Power_Management.kicad_sch (KiCad schematic)
At the start: 14 parts, among them IC4 LMR33630ADDA

Commit message: Use shared Kicad_Libs instead of project-specific libraries
- Project parts moved to Kicad_Libs (symbol, footprint, 3D, datasheet)
- Lib tables point to ${KIPRJMOD}/../KiCad_Libs (link via bring_libs.bat)
- Schematic/PCB references (lib ids, footprints, 3D paths, datasheets)
  updated to the Kicad_Libs libraries; no design changes
- Removed the old project-specific library folder
Parts:
- IC4: footprint SOIC127P600X170-9N -> eConverterDCDC:SOIC127P600X170-9N; symbol LMR33630BDDA:LMR33630BDDA -> eConverterDCDC:LMR33630BDDA
- L5: footprint IHLP2525CZER6R8M8A:INDPM6965X300N -> eCoil:INDPM6965X300N; symbol IHLP2525CZER6R8M8A:IHLP2525CZER6R8M8A -> eCoil:IHLP2525CZER6R8M8A
Changed lines of the file:
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@@
 	)
 	(symbol
-		(lib_id "IHLP2525CZER6R8M8A:IHLP2525CZER6R8M8A")
+		(lib_id "eCoil:IHLP2525CZER6R8M8A")
 		(at 139.7 77.47 0)
 		(unit 1)
@@
 			)
 		)
-		(property "Footprint" "IHLP2525CZER6R8M8A:INDPM6965X300N"
+		(property "Footprint" "eCoil:INDPM6965X300N"
 			(at 156.21 173.66 0)
 			(hide yes)
@@
 			)
 		)
-		(property "Datasheet" "kicad-embed://ihlp-2525cz-8a.pdf"
+		(property "Datasheet" "${KIPRJMOD}/../KiCad_Libs/eCoil/datasheet/ihlp-2525cz-8a.pdf"
 			(at 156.21 273.66 0)
 			(hide yes)
@@
 	)
 	(symbol
-		(lib_id "LMR33630BDDA:LMR33630BDDA")
+		(lib_id "eConverterDCDC:LMR33630BDDA")
 		(at 95.25 76.2 0)
 		(unit 1)
@@
 			)
 		)
-		(property "Footprint" "SOIC127P600X170-9N"
+		(property "Footprint" "eConverterDCDC:SOIC127P600X170-9N"
 			(at 121.92 171.12 0)
 			(hide yes)
@@
 			)
 		)
-		(property "Datasheet" "http://www.ti.com/lit/gpn/LMR33630"
+		(property "Datasheet" "${KIPRJMOD}/../KiCad_Libs/eConverterDCDC/datasheet/lmr33630.pdf"
 			(at 121.92 271.12 0)
 			(hide yes)
