File: KiCad_Project/Audio_Amp_BT/02_Bluetooth_Receiver.kicad_sch (KiCad schematic)
At the start: 12 parts, among them IC3 BM64SPKS1MC2-0002AA

Commit message: Use shared Kicad_Libs instead of project-specific libraries
- Project parts moved to Kicad_Libs (symbol, footprint, 3D, datasheet)
- Lib tables point to ${KIPRJMOD}/../KiCad_Libs (link via bring_libs.bat)
- Schematic/PCB references (lib ids, footprints, 3D paths, datasheets)
  updated to the Kicad_Libs libraries; no design changes
- Removed the old project-specific library folder
Parts:
- IC3: footprint BM64SPKS1MC20002AA -> eRFModule:BM64SPKS1MC20002AA; symbol BM64SPKS1MC2-0002AA:BM64SPKS1MC2-0002AA -> eRFModule:BM64SPKS1MC2-0002AA
Changed lines of the file:
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@@
 	)
 	(symbol
-		(lib_id "BM64SPKS1MC2-0002AA:BM64SPKS1MC2-0002AA")
+		(lib_id "eRFModule:BM64SPKS1MC2-0002AA")
 		(at 123.19 60.96 0)
 		(unit 1)
@@
 			)
 		)
-		(property "Footprint" "BM64SPKS1MC20002AA"
+		(property "Footprint" "eRFModule:BM64SPKS1MC20002AA"
 			(at 157.48 155.88 0)
 			(hide yes)
@@
 			)
 		)
-		(property "Datasheet" "kicad-embed://BM62-64-Bluetooth-Stereo-Audio-Module-DS60001403.pdf"
+		(property "Datasheet" "${KIPRJMOD}/../KiCad_Libs/eRFModule/datasheet/BM62-64-Bluetooth-Stereo-Audio-Module-DS60001403.pdf"
 			(at 157.48 255.88 0)
 			(hide yes)
