File: KiCad_Project/Audio_Amp_BT/03_Audio_DAC.kicad_sch (KiCad schematic)
At the start: 25 parts, among them U1 PCM2704CDB, Y1 ABM8-12.000MHZ-12-B1U-T

Commit message: Use shared Kicad_Libs instead of project-specific libraries
- Project parts moved to Kicad_Libs (symbol, footprint, 3D, datasheet)
- Lib tables point to ${KIPRJMOD}/../KiCad_Libs (link via bring_libs.bat)
- Schematic/PCB references (lib ids, footprints, 3D paths, datasheets)
  updated to the Kicad_Libs libraries; no design changes
- Removed the old project-specific library folder
Parts:
- U1: footprint PCM2704CDB:SOP65P780X200-28N -> eConverterADDA:SOP65P780X200-28N; symbol PCM2704CDB:PCM2704CDB -> eConverterADDA:PCM2704CDB
- Y1: footprint ABM810000MHZ12D2W -> eCrystal:ABM810000MHZ12D2W; symbol ABM8-12_000MHZ-12-B1U-T:ABM8-12.000MHZ-12-B1U-T -> eCrystal:ABM8-12.000MHZ-12-B1U-T
Changed lines of the file:
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@@
 	)
 	(symbol
-		(lib_id "PCM2704CDB:PCM2704CDB")
+		(lib_id "eConverterADDA:PCM2704CDB")
 		(at 134.62 97.79 0)
 		(unit 1)
@@
 			)
 		)
-		(property "Footprint" "PCM2704CDB:SOP65P780X200-28N"
+		(property "Footprint" "eConverterADDA:SOP65P780X200-28N"
 			(at 134.62 97.79 0)
 			(hide yes)
@@
 			)
 		)
-		(property "Datasheet" "kicad-embed://pcm2704c.pdf"
+		(property "Datasheet" "${KIPRJMOD}/../KiCad_Libs/eConverterADDA/datasheet/pcm2704c.pdf"
 			(at 134.62 97.79 0)
 			(hide yes)
@@
 	)
 	(symbol
-		(lib_id "ABM8-12_000MHZ-12-B1U-T:ABM8-12.000MHZ-12-B1U-T")
+		(lib_id "eCrystal:ABM8-12.000MHZ-12-B1U-T")
 		(at 116.84 50.8 0)
 		(unit 1)
@@
 			)
 		)
-		(property "Footprint" "ABM810000MHZ12D2W"
+		(property "Footprint" "eCrystal:ABM810000MHZ12D2W"
 			(at 143.51 145.72 0)
 			(hide yes)
@@
 			)
 		)
-		(property "Datasheet" "https://abracon.com/Resonators/abm8.pdf"
+		(property "Datasheet" "${KIPRJMOD}/../KiCad_Libs/eCrystal/datasheet/abm8.pdf"
 			(at 143.51 245.72 0)
 			(hide yes)
