File: KiCad_Project/Audio_Amp_BT/05_Power_Amplifier.kicad_sch (KiCad schematic)
At the start: 43 parts, among them IC2 TPA3116D2DAD

Commit message: Use shared Kicad_Libs instead of project-specific libraries
- Project parts moved to Kicad_Libs (symbol, footprint, 3D, datasheet)
- Lib tables point to ${KIPRJMOD}/../KiCad_Libs (link via bring_libs.bat)
- Schematic/PCB references (lib ids, footprints, 3D paths, datasheets)
  updated to the Kicad_Libs libraries; no design changes
- Removed the old project-specific library folder
Parts:
- C10, C17: footprint EEE-FK1H221GV:EEHZT1E561UV -> eCapacitor:EEHZT1E561UV
- IC2: footprint TPA3116D2DAD:SOP65P810X120-32N -> eAmplifier:SOP65P810X120-32N; symbol TPA3116D2DAD:TPA3116D2DAD -> eAmplifier:TPA3116D2DAD
- L1, L2, L3, L4: footprint 7443341000:INDPM8479X720N -> eCoil:INDPM8479X720N
Changed lines of the file:
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@@
 			)
 		)
-		(property "Footprint" "7443341000:INDPM8479X720N"
+		(property "Footprint" "eCoil:INDPM8479X720N"
 			(at 181.61 149.86 0)
 			(hide yes)
@@
 			)
 		)
-		(property "Datasheet" "kicad-embed://7443341000.pdf"
+		(property "Datasheet" "${KIPRJMOD}/../KiCad_Libs/eCoil/datasheet/7443341000.pdf"
 			(at 181.61 149.86 0)
 			(hide yes)
@@
 			)
 		)
-		(property "Footprint" "EEE-FK1H221GV:EEHZT1E561UV"
+		(property "Footprint" "eCapacitor:EEHZT1E561UV"
 			(at 163.83 143.51 0)
 			(hide yes)
@@
 			)
 		)
-		(property "Datasheet" "kicad-embed://ABA0000C1181.pdf"
+		(property "Datasheet" "${KIPRJMOD}/../KiCad_Libs/eCapacitor/datasheet/ABA0000C1181.pdf"
 			(at 163.83 143.51 0)
 			(hide yes)
@@
 			)
 		)
-		(property "Footprint" "7443341000:INDPM8479X720N"
+		(property "Footprint" "eCoil:INDPM8479X720N"
 			(at 181.61 90.17 0)
 			(hide yes)
@@
 			)
 		)
-		(property "Datasheet" "kicad-embed://7443341000.pdf"
+		(property "Datasheet" "${KIPRJMOD}/../KiCad_Libs/eCoil/datasheet/7443341000.pdf"
 			(at 181.61 90.17 0)
 			(hide yes)
@@
 			)
 		)
-		(property "Footprint" "EEE-FK1H221GV:EEHZT1E561UV"
+		(property "Footprint" "eCapacitor:EEHZT1E561UV"
 			(at 165.1 46.99 0)
 			(hide yes)
@@
 			)
 		)
-		(property "Datasheet" "kicad-embed://ABA0000C1181.pdf"
+		(property "Datasheet" "${KIPRJMOD}/../KiCad_Libs/eCapacitor/datasheet/ABA0000C1181.pdf"
 			(at 165.1 46.99 0)
 			(hide yes)
@@
 	)
 	(symbol
-		(lib_id "TPA3116D2DAD:TPA3116D2DAD")
+		(lib_id "eAmplifier:TPA3116D2DAD")
 		(at 95.25 92.71 0)
 		(unit 1)
@@
 			)
 		)
-		(property "Footprint" "TPA3116D2DAD:SOP65P810X120-32N"
+		(property "Footprint" "eAmplifier:SOP65P810X120-32N"
 			(at 127 187.63 0)
 			(hide yes)
@@
 			)
 		)
-		(property "Datasheet" "kicad-embed://tpa3116d2.pdf"
+		(property "Datasheet" "${KIPRJMOD}/../KiCad_Libs/eAmplifier/datasheet/tpa3116d2.pdf"
 			(at 127 287.63 0)
 			(hide yes)
@@
 			)
 		)
-		(property "Footprint" "7443341000:INDPM8479X720N"
+		(property "Footprint" "eCoil:INDPM8479X720N"
 			(at 181.61 101.6 0)
 			(hide yes)
@@
 			)
 		)
-		(property "Datasheet" "kicad-embed://7443341000.pdf"
+		(property "Datasheet" "${KIPRJMOD}/../KiCad_Libs/eCoil/datasheet/7443341000.pdf"
 			(at 181.61 101.6 0)
 			(hide yes)
@@
 			)
 		)
-		(property "Footprint" "7443341000:INDPM8479X720N"
+		(property "Footprint" "eCoil:INDPM8479X720N"
 			(at 181.61 41.91 0)
 			(hide yes)
@@
 			)
 		)
-		(property "Datasheet" "kicad-embed://7443341000.pdf"
+		(property "Datasheet" "${KIPRJMOD}/../KiCad_Libs/eCoil/datasheet/7443341000.pdf"
 			(at 181.61 41.91 0)
 			(hide yes)
