File: KiCad_Project/Audio_Amp_BT/06_Connectors_IO.kicad_sch (KiCad schematic)
At the start: 4 parts, among them J1 TS-103-T-A, J2 1729128, J3 1729128, J4 PJ-102AH

Commit message: Use shared Kicad_Libs instead of project-specific libraries
- Project parts moved to Kicad_Libs (symbol, footprint, 3D, datasheet)
- Lib tables point to ${KIPRJMOD}/../KiCad_Libs (link via bring_libs.bat)
- Schematic/PCB references (lib ids, footprints, 3D paths, datasheets)
  updated to the Kicad_Libs libraries; no design changes
- Removed the old project-specific library folder
Parts:
- J1: footprint TS_103_T_A:SAMTEC_TS-103-T-A -> eConnector:SAMTEC_TS-103-T-A; symbol TS-103-T-A:TS-103-T-A -> eConnector:TS-103-T-A
- J2, J3: footprint 1729128 -> eConnector:1729128; symbol 1729128:1729128 -> eConnector:1729128
- J4: footprint PJ-102AH -> eConnector:PJ-102AH; symbol PJ-102AH:PJ-102AH -> eConnector:PJ-102AH
Changed lines of the file:
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@@
 	)
 	(symbol
-		(lib_id "TS-103-T-A:TS-103-T-A")
+		(lib_id "eConnector:TS-103-T-A")
 		(at 36.83 116.84 180)
 		(unit 1)
@@
 			)
 		)
-		(property "Footprint" "TS_103_T_A:SAMTEC_TS-103-T-A"
+		(property "Footprint" "eConnector:SAMTEC_TS-103-T-A"
 			(at 36.83 116.84 0)
 			(hide yes)
@@
 			)
 		)
-		(property "Datasheet" "kicad-embed://td.pdf"
+		(property "Datasheet" "${KIPRJMOD}/../KiCad_Libs/eConnector/datasheet/Samtec_TS-103-T-A.pdf"
 			(at 36.83 116.84 0)
 			(hide yes)
@@
 	)
 	(symbol
-		(lib_id "1729128:1729128")
+		(lib_id "eConnector:1729128")
 		(at 115.57 96.52 0)
 		(unit 1)
@@
 			)
 		)
-		(property "Footprint" "1729128"
+		(property "Footprint" "eConnector:1729128"
 			(at 132.08 191.44 0)
 			(hide yes)
@@
 			)
 		)
-		(property "Datasheet" "kicad-embed://phoenix_contact_1729128_en.pdf"
+		(property "Datasheet" "${KIPRJMOD}/../KiCad_Libs/eConnector/datasheet/phoenix_contact_1729128_en.pdf"
 			(at 132.08 291.44 0)
 			(hide yes)
@@
 	)
 	(symbol
-		(lib_id "1729128:1729128")
+		(lib_id "eConnector:1729128")
 		(at 115.57 81.28 0)
 		(unit 1)
@@
 			)
 		)
-		(property "Footprint" "1729128"
+		(property "Footprint" "eConnector:1729128"
 			(at 132.08 176.2 0)
 			(hide yes)
@@
 			)
 		)
-		(property "Datasheet" "kicad-embed://phoenix_contact_1729128_en.pdf"
+		(property "Datasheet" "${KIPRJMOD}/../KiCad_Libs/eConnector/datasheet/phoenix_contact_1729128_en.pdf"
 			(at 132.08 276.2 0)
 			(hide yes)
@@
 	)
 	(symbol
-		(lib_id "PJ-102AH:PJ-102AH")
+		(lib_id "eConnector:PJ-102AH")
 		(at 29.21 95.25 0)
 		(unit 1)
@@
 			)
 		)
-		(property "Footprint" "PJ-102AH"
+		(property "Footprint" "eConnector:PJ-102AH"
 			(at 45.72 190.17 0)
 			(hide yes)
@@
 			)
 		)
-		(property "Datasheet" "https://www.sameskydevices.com/product/resource/pj-102ah.pdf"
+		(property "Datasheet" "${KIPRJMOD}/../KiCad_Libs/eConnector/datasheet/pj_102ah.pdf"
 			(at 45.72 290.17 0)
 			(hide yes)
