File: KiCad_Project/Audio_Amp_BT/Audio_Amp_v1.kicad_pcb (KiCad board)
At the start: 2 copper layers, 93.5 x 52.8 mm, 73 parts, among them IC2 TPA3116D2DAD, IC3 BM64SPKS1MC2-0002AA, IC4 LMR33630ADDA, J1 TS-103-T-A, J2 1729128, J3 1729128, J4 PJ-102AH

Commit message: Use shared Kicad_Libs instead of project-specific libraries
- Project parts moved to Kicad_Libs (symbol, footprint, 3D, datasheet)
- Lib tables point to ${KIPRJMOD}/../KiCad_Libs (link via bring_libs.bat)
- Schematic/PCB references (lib ids, footprints, 3D paths, datasheets)
  updated to the Kicad_Libs libraries; no design changes
- Removed the old project-specific library folder
Parts:
- C10, C17: footprint EEE-FK1H221GV:EEHZT1E561UV -> eCapacitor:EEHZT1E561UV
- IC2: footprint TPA3116D2DAD:SOP65P810X120-32N -> eAmplifier:SOP65P810X120-32N
- IC3: footprint Bluetooth_Module:BM64SPKS1MC20002AA -> eRFModule:BM64SPKS1MC20002AA
- IC4: footprint LMR33630:SOIC127P600X170-9N -> eConverterDCDC:SOIC127P600X170-9N
- J1: footprint TS_103_T_A:SAMTEC_TS-103-T-A -> eConnector:SAMTEC_TS-103-T-A
- J2, J3: footprint Phoenix-1729128:1729128 -> eConnector:1729128
- J4: footprint 24V-JACK:PJ-102AH -> eConnector:PJ-102AH
- L1, L2, L3, L4: footprint 7443341000:INDPM8479X720N -> eCoil:INDPM8479X720N
- L5: footprint IHLP2525CZER6R8M8A:INDPM6965X300N -> eCoil:INDPM6965X300N
Changed lines of the file:
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@@
 		)
 	)
-	(footprint "IHLP2525CZER6R8M8A:INDPM6965X300N"
+	(footprint "eCoil:INDPM6965X300N"
 		(layer "F.Cu")
 		(at 98.75 85.25 180)
@@
 			)
 		)
-		(property "Datasheet" "kicad-embed://ihlp-2525cz-8a.pdf"
+		(property "Datasheet" "${KIPRJMOD}/../KiCad_Libs/eCoil/datasheet/ihlp-2525cz-8a.pdf"
 			(at 0 0 0)
 			(layer "F.Fab")
@@
 		)
 		(embedded_fonts no)
-		(model "IHLP2525CZER6R8M8A.stp"
+		(model "${KIPRJMOD}/../KiCad_Libs/eCoil/eCoil.3dshapes/IHLP2525CZER6R8M8A.stp"
 			(offset
 				(xyz -1.499999977 5.300000111 -2.400000059)
@@
 		)
 	)
-	(footprint "TPA3116D2DAD:SOP65P810X120-32N"
+	(footprint "eAmplifier:SOP65P810X120-32N"
 		(layer "F.Cu")
 		(at 118.5 108.5)
@@
 			)
 		)
-		(property "Datasheet" "kicad-embed://tpa3116d2.pdf"
+		(property "Datasheet" "${KIPRJMOD}/../KiCad_Libs/eAmplifier/datasheet/tpa3116d2.pdf"
 			(at 0 0 0)
 			(layer "F.Fab")
@@
 		)
 		(embedded_fonts no)
-		(model "TPA3116D2DAD.stp"
+		(model "${KIPRJMOD}/../KiCad_Libs/eAmplifier/eAmplifier.3dshapes/TPA3116D2DAD.stp"
 			(offset
 				(xyz 0 0 0)
@@
 		)
 	)
-	(footprint "7443341000:INDPM8479X720N"
+	(footprint "eCoil:INDPM8479X720N"
 		(layer "F.Cu")
 		(at 136.288 113.625)
@@
 			)
 		)
-		(property "Datasheet" "kicad-embed://7443341000.pdf"
+		(property "Datasheet" "${KIPRJMOD}/../KiCad_Libs/eCoil/datasheet/7443341000.pdf"
 			(at 0 0 0)
 			(layer "F.Fab")
@@
 		)
 		(embedded_fonts no)
-		(model "7443341000.stp"
+		(model "${KIPRJMOD}/../KiCad_Libs/eCoil/eCoil.3dshapes/7443341000.stp"
 			(offset
 				(xyz 0 0 0.04999999999)
@@
 		)
 	)
-	(footprint "Phoenix-1729128:1729128"
+	(footprint "eConnector:1729128"
 		(layer "F.Cu")
 		(at 157 116.5 -90)
@@
 			)
 		)
-		(property "Datasheet" "kicad-embed://phoenix_contact_1729128_en.pdf"
+		(property "Datasheet" "${KIPRJMOD}/../KiCad_Libs/eConnector/datasheet/phoenix_contact_1729128_en.pdf"
 			(at 0 0 90)
 			(layer "F.Fab")
@@
 		)
 		(embedded_fonts no)
-		(model "1729128.stp"
+		(model "${KIPRJMOD}/../KiCad_Libs/eConnector/eConnector.3dshapes/1729128.stp"
 			(offset
 				(xyz -2.609999856 -4.070000111 0)
@@
 		)
 	)
-	(footprint "24V-JACK:PJ-102AH"
+	(footprint "eConnector:PJ-102AH"
 		(layer "F.Cu")
 		(at 76.515075 98.85 90)
@@
 			)
 		)
-		(property "Datasheet" "https://www.sameskydevices.com/product/resource/pj-102ah.pdf"
+		(property "Datasheet" "${KIPRJMOD}/../KiCad_Libs/eConnector/datasheet/pj_102ah.pdf"
 			(at 0 0 90)
 			(layer "F.Fab")
@@
 		)
 		(embedded_fonts no)
-		(model "PJ-102AH.stp"
+		(model "${KIPRJMOD}/../KiCad_Libs/eConnector/eConnector.3dshapes/PJ-102AH.stp"
 			(offset
 				(xyz 4.159999785 10.64999946 6.269999887)
@@
 		)
 	)
-	(footprint "EEE-FK1H221GV:EEHZT1E561UV"
+	(footprint "eCapacitor:EEHZT1E561UV"
 		(layer "F.Cu")
 		(at 115.788 121.875 -90)
@@
 			)
 		)
-		(property "Datasheet" "kicad-embed://ABA0000C1181.pdf"
+		(property "Datasheet" "${KIPRJMOD}/../KiCad_Libs/eCapacitor/datasheet/ABA0000C1181.pdf"
 			(at 0 0 90)
 			(layer "F.Fab")
@@
 		)
 		(embedded_fonts no)
-		(model "EEE-FK1H221GV.stp"
+		(model "${KIPRJMOD}/../KiCad_Libs/eCapacitor/eCapacitor.3dshapes/EEE-FK1H221GV.stp"
 			(offset
 				(xyz 0 0 0.999999985)
@@
 		)
 	)
-	(footprint "7443341000:INDPM8479X720N"
+	(footprint "eCoil:INDPM8479X720N"
 		(layer "F.Cu")
 		(at 136.288 122.875)
@@
 			)
 		)
-		(property "Datasheet" "kicad-embed://7443341000.pdf"
+		(property "Datasheet" "${KIPRJMOD}/../KiCad_Libs/eCoil/datasheet/7443341000.pdf"
 			(at 0 0 0)
 			(layer "F.Fab")
@@
 		)
 		(embedded_fonts no)
-		(model "7443341000.stp"
+		(model "${KIPRJMOD}/../KiCad_Libs/eCoil/eCoil.3dshapes/7443341000.stp"
 			(offset
 				(xyz 0 0 0.04999999999)
@@
 		)
 	)
-	(footprint "EEE-FK1H221GV:EEHZT1E561UV"
+	(footprint "eCapacitor:EEHZT1E561UV"
 		(layer "F.Cu")
 		(at 116.988 88.325 -90)
@@
 			)
 		)
-		(property "Datasheet" "kicad-embed://ABA0000C1181.pdf"
+		(property "Datasheet" "${KIPRJMOD}/../KiCad_Libs/eCapacitor/datasheet/ABA0000C1181.pdf"
 			(at 0 0 90)
 			(layer "F.Fab")
@@
 		)
 		(embedded_fonts no)
-		(model "EEE-FK1H221GV.stp"
+		(model "${KIPRJMOD}/../KiCad_Libs/eCapacitor/eCapacitor.3dshapes/EEE-FK1H221GV.stp"
 			(offset
 				(xyz 0 0 0.999999985)
@@
 		)
 	)
-	(footprint "7443341000:INDPM8479X720N"
+	(footprint "eCoil:INDPM8479X720N"
 		(layer "F.Cu")
 		(at 136.288 104.125 180)
@@
 			)
 		)
-		(property "Datasheet" "kicad-embed://7443341000.pdf"
+		(property "Datasheet" "${KIPRJMOD}/../KiCad_Libs/eCoil/datasheet/7443341000.pdf"
 			(at 0 0 0)
 			(layer "F.Fab")
@@
 		)
 		(embedded_fonts no)
-		(model "7443341000.stp"
+		(model "${KIPRJMOD}/../KiCad_Libs/eCoil/eCoil.3dshapes/7443341000.stp"
 			(offset
 				(xyz 0 0 0.04999999999)
@@
 		)
 	)
-	(footprint "7443341000:INDPM8479X720N"
+	(footprint "eCoil:INDPM8479X720N"
 		(layer "F.Cu")
 		(at 136.188 94.875)
@@
 			)
 		)
-		(property "Datasheet" "kicad-embed://7443341000.pdf"
+		(property "Datasheet" "${KIPRJMOD}/../KiCad_Libs/eCoil/datasheet/7443341000.pdf"
 			(at 0 0 0)
 			(layer "F.Fab")
@@
 		)
 		(embedded_fonts no)
-		(model "7443341000.stp"
+		(model "${KIPRJMOD}/../KiCad_Libs/eCoil/eCoil.3dshapes/7443341000.stp"
 			(offset
 				(xyz 0 0 0.04999999999)
@@
 		)
 	)
-	(footprint "Bluetooth_Module:BM64SPKS1MC20002AA"
+	(footprint "eRFModule:BM64SPKS1MC20002AA"
 		(layer "F.Cu")
 		(at 78.1 116.25 90)
@@
 			)
 		)
-		(property "Datasheet" "kicad-embed://BM62-64-Bluetooth-Stereo-Audio-Module-DS60001403.pdf"
+		(property "Datasheet" "${KIPRJMOD}/../KiCad_Libs/eRFModule/datasheet/BM62-64-Bluetooth-Stereo-Audio-Module-DS60001403.pdf"
 			(at 0 0 90)
 			(layer "F.Fab")
@@
 		)
 		(embedded_fonts no)
-		(model "BM64SPKS1MC2-0002AA.stp"
+		(model "${KIPRJMOD}/../KiCad_Libs/eRFModule/eRFModule.3dshapes/BM64SPKS1MC2-0002AA.stp"
 			(offset
 				(xyz 0 0 0)
@@
 		)
 	)
-	(footprint "Phoenix-1729128:1729128"
+	(footprint "eConnector:1729128"
 		(layer "F.Cu")
 		(at 156.75 97.67 -90)
@@
 			)
 		)
-		(property "Datasheet" "kicad-embed://phoenix_contact_1729128_en.pdf"
+		(property "Datasheet" "${KIPRJMOD}/../KiCad_Libs/eConnector/datasheet/phoenix_contact_1729128_en.pdf"
 			(at 0 0 90)
 			(layer "F.Fab")
@@
 		)
 		(embedded_fonts no)
-		(model "1729128.stp"
+		(model "${KIPRJMOD}/../KiCad_Libs/eConnector/eConnector.3dshapes/1729128.stp"
 			(offset
 				(xyz -2.609999856 -4.070000111 0)
@@
 		)
 	)
-	(footprint "LMR33630:SOIC127P600X170-9N"
+	(footprint "eConverterDCDC:SOIC127P600X170-9N"
 		(layer "F.Cu")
 		(at 98.75 92.865)
@@
 			)
 		)
-		(property "Datasheet" "http://www.ti.com/lit/gpn/LMR33630"
+		(property "Datasheet" "${KIPRJMOD}/../KiCad_Libs/eConverterDCDC/datasheet/lmr33630.pdf"
 			(at 0 0 0)
 			(layer "F.Fab")
@@
 		)
 		(embedded_fonts no)
-		(model "LMR33630BDDA.stp"
+		(model "${KIPRJMOD}/../KiCad_Libs/eConverterDCDC/eConverterDCDC.3dshapes/LMR33630BDDA.stp"
 			(offset
 				(xyz 0 0 0)
@@
 		)
 	)
-	(footprint "TS_103_T_A:SAMTEC_TS-103-T-A"
+	(footprint "eConnector:SAMTEC_TS-103-T-A"
 		(layer "F.Cu")
 		(at 100.75 128.25)
@@
 			)
 		)
-		(property "Datasheet" "kicad-embed://td.pdf"
+		(property "Datasheet" "${KIPRJMOD}/../KiCad_Libs/eConnector/datasheet/Samtec_TS-103-T-A.pdf"
 			(at 0 0 0)
 			(layer "F.Fab")
